Commit message: Bicolor hermes arm visualization

File: hermes_arm_kdl/urdf/hermesArm.urdf (robot description, URDF)
Before this commit: robot hermesArm, 8 links, 7 joints
Links:
- link base: mass None -> 1.0; geometry collision mesh filename=package://hermes_arm_kdl/stl/BaseSchunkLow.stl; visual mesh filename=package://hermes_arm_kdl/stl/BaseSchunk.stl
- link link1: mass None -> 1.0; geometry collision mesh filename=package://hermes_arm_kdl/stl/SchunkLink1Low.stl; visual mesh filename=package://hermes_arm_kdl/stl/SchunkLink1.stl
- link link2: mass None -> 1.0; geometry collision mesh filename=package://hermes_arm_kdl/stl/SchunkLink2Low.stl; visual mesh filename=package://hermes_arm_kdl/stl/SchunkLink2.stl
- link link3: mass None -> 1.0; geometry collision mesh filename=package://hermes_arm_kdl/stl/SchunkLink3Low.stl; visual mesh filename=package://hermes_arm_kdl/stl/SchunkLink3.stl
- link link4: mass None -> 1.0; geometry collision mesh filename=package://hermes_arm_kdl/stl/SchunkLink4Low.stl; visual mesh filename=package://hermes_arm_kdl/stl/SchunkLink4.stl
- link link5: mass None -> 1.0; geometry collision mesh filename=package://hermes_arm_kdl/stl/SchunkLink5Low.stl; visual mesh filename=package://hermes_arm_kdl/stl/SchunkLink5.stl
- link link6: mass None -> 1.0; geometry collision mesh filename=package://hermes_arm_kdl/stl/SchunkLink6Low.stl; visual mesh filename=package://hermes_arm_kdl/stl/SchunkLink6.stl
- link link7: mass None -> 1.0; geometry collision mesh filename=package://hermes_arm_kdl/stl/SchunkLink7Low.stl; visual mesh filename=package://hermes_arm_kdl/stl/SchunkLink7.stl

Commit message: Model hermes arm multicolor

File: hermes_arm_kdl/urdf/hermesArm.urdf (robot description, URDF)
Before this commit: robot hermesArm, 8 links, 7 joints
Links:
- removed link base
- removed link link1
- removed link link2
- removed link link3
- removed link link4
- removed link link5
- removed link link6
- removed link link7
- added link base1, mass 1.0; collision mesh filename=package://hermes_arm_kdl/stl/BaseSchunk1.stl; visual mesh filename=package://hermes_arm_kdl/stl/BaseSchunk1.stl
- added link base2, mass 1.0; collision mesh filename=package://hermes_arm_kdl/stl/BaseSchunk2.stl; visual mesh filename=package://hermes_arm_kdl/stl/BaseSchunk2.stl
- added link link1_1, mass 1.0; collision mesh filename=package://hermes_arm_kdl/stl/SchunkLink1_1.stl; visual mesh filename=package://hermes_arm_kdl/stl/SchunkLink1_1.stl
- added link link1_2, mass 1.0; collision mesh filename=package://hermes_arm_kdl/stl/SchunkLink1_2.stl; visual mesh filename=package://hermes_arm_kdl/stl/SchunkLink1_2.stl
- added link link1_3, mass 1.0; collision mesh filename=package://hermes_arm_kdl/stl/SchunkLink1_3.stl; visual mesh filename=package://hermes_arm_kdl/stl/SchunkLink1_3.stl
- added link link1_4, mass 1.0; collision mesh filename=package://hermes_arm_kdl/stl/SchunkLink1_4.stl; visual mesh filename=package://hermes_arm_kdl/stl/SchunkLink1_4.stl
- added link link1_5, mass 1.0; collision mesh filename=package://hermes_arm_kdl/stl/SchunkLink1_5.stl; visual mesh filename=package://hermes_arm_kdl/stl/SchunkLink1_5.stl
- added link link2_1, mass 1.0; collision mesh filename=package://hermes_arm_kdl/stl/SchunkLink2_1.stl; visual mesh filename=package://hermes_arm_kdl/stl/SchunkLink2_1.stl
- added link link2_2, mass 1.0; collision mesh filename=package://hermes_arm_kdl/stl/SchunkLink2_2.stl; visual mesh filename=package://hermes_arm_kdl/stl/SchunkLink2_2.stl
- added link link2_3, mass 1.0; collision mesh filename=package://hermes_arm_kdl/stl/SchunkLink2_3.stl; visual mesh filename=package://hermes_arm_kdl/stl/SchunkLink2_3.stl
- added link link2_4, mass 1.0; collision mesh filename=package://hermes_arm_kdl/stl/SchunkLink2_4.stl; visual mesh filename=package://hermes_arm_kdl/stl/SchunkLink2_4.stl
- added link link2_5, mass 1.0; collision mesh filename=package://hermes_arm_kdl/stl/SchunkLink2_5.stl; visual mesh filename=package://hermes_arm_kdl/stl/SchunkLink2_5.stl
- added link link3_1, mass 1.0; collision mesh filename=package://hermes_arm_kdl/stl/SchunkLink3_1.stl; visual mesh filename=package://hermes_arm_kdl/stl/SchunkLink3_1.stl
- added link link3_2, mass 1.0; collision mesh filename=package://hermes_arm_kdl/stl/SchunkLink3_2.stl; visual mesh filename=package://hermes_arm_kdl/stl/SchunkLink3_2.stl
- added link link3_3, mass 1.0; collision mesh filename=package://hermes_arm_kdl/stl/SchunkLink3_3.stl; visual mesh filename=package://hermes_arm_kdl/stl/SchunkLink3_3.stl
- added link link3_4, mass 1.0; collision mesh filename=package://hermes_arm_kdl/stl/SchunkLink3_4.stl; visual mesh filename=package://hermes_arm_kdl/stl/SchunkLink3_4.stl
- added link link3_5, mass 1.0; collision mesh filename=package://hermes_arm_kdl/stl/SchunkLink3_5.stl; visual mesh filename=package://hermes_arm_kdl/stl/SchunkLink3_5.stl
- added link link4_1, mass 1.0; collision mesh filename=package://hermes_arm_kdl/stl/SchunkLink4_1.stl; visual mesh filename=package://hermes_arm_kdl/stl/SchunkLink4_1.stl
- added link link4_2, mass 1.0; collision mesh filename=package://hermes_arm_kdl/stl/SchunkLink4_2.stl; visual mesh filename=package://hermes_arm_kdl/stl/SchunkLink4_2.stl
- added link link4_3, mass 1.0; collision mesh filename=package://hermes_arm_kdl/stl/SchunkLink4_3.stl; visual mesh filename=package://hermes_arm_kdl/stl/SchunkLink4_3.stl
- added link link4_4, mass 1.0; collision mesh filename=package://hermes_arm_kdl/stl/SchunkLink4_4.stl; visual mesh filename=package://hermes_arm_kdl/stl/SchunkLink4_4.stl
- added link link4_5, mass 1.0; collision mesh filename=package://hermes_arm_kdl/stl/SchunkLink4_5.stl; visual mesh filename=package://hermes_arm_kdl/stl/SchunkLink4_5.stl
- added link link5_1, mass 1.0; collision mesh filename=package://hermes_arm_kdl/stl/SchunkLink5_1.stl; visual mesh filename=package://hermes_arm_kdl/stl/SchunkLink5_1.stl
- added link link5_2, mass 1.0; collision mesh filename=package://hermes_arm_kdl/stl/SchunkLink5_2.stl; visual mesh filename=package://hermes_arm_kdl/stl/SchunkLink5_2.stl
- added link link5_3, mass 1.0; collision mesh filename=package://hermes_arm_kdl/stl/SchunkLink5_3.stl; visual mesh filename=package://hermes_arm_kdl/stl/SchunkLink5_3.stl
- added link link5_4, mass 1.0; collision mesh filename=package://hermes_arm_kdl/stl/SchunkLink5_4.stl; visual mesh filename=package://hermes_arm_kdl/stl/SchunkLink5_4.stl
- added link link5_5, mass 1.0; collision mesh filename=package://hermes_arm_kdl/stl/SchunkLink5_5.stl; visual mesh filename=package://hermes_arm_kdl/stl/SchunkLink5_5.stl
- added link link6_1, mass 1.0; collision mesh filename=package://hermes_arm_kdl/stl/SchunkLink6_1.stl; visual mesh filename=package://hermes_arm_kdl/stl/SchunkLink6_1.stl
- added link link6_2, mass 1.0; collision mesh filename=package://hermes_arm_kdl/stl/SchunkLink6_2.stl; visual mesh filename=package://hermes_arm_kdl/stl/SchunkLink6_2.stl
- added link link6_3, mass 1.0; collision mesh filename=package://hermes_arm_kdl/stl/SchunkLink6_3.stl; visual mesh filename=package://hermes_arm_kdl/stl/SchunkLink6_3.stl
- added link link6_4, mass 1.0; collision mesh filename=package://hermes_arm_kdl/stl/SchunkLink6_4.stl; visual mesh filename=package://hermes_arm_kdl/stl/SchunkLink6_4.stl
- added link link6_5, mass 1.0; collision mesh filename=package://hermes_arm_kdl/stl/SchunkLink6_5.stl; visual mesh filename=package://hermes_arm_kdl/stl/SchunkLink6_5.stl
- added link link7_1, mass 1.0; collision mesh filename=package://hermes_arm_kdl/stl/SchunkLink7_1.stl; visual mesh filename=package://hermes_arm_kdl/stl/SchunkLink7_1.stl
- added link link7_2, mass 1.0; collision mesh filename=package://hermes_arm_kdl/stl/SchunkLink7_2.stl; visual mesh filename=package://hermes_arm_kdl/stl/SchunkLink7_2.stl
- added link link7_3, mass 1.0; collision mesh filename=package://hermes_arm_kdl/stl/SchunkLink7_3.stl; visual mesh filename=package://hermes_arm_kdl/stl/SchunkLink7_3.stl
- added link link7_4, mass 1.0; collision mesh filename=package://hermes_arm_kdl/stl/SchunkLink7_4.stl; visual mesh filename=package://hermes_arm_kdl/stl/SchunkLink7_4.stl
Joints:
- added joint base_fixed: type fixed, parent base1, child base2
- added joint joint1_1: type fixed, parent link1_1, child link1_2
- added joint joint1_2: type fixed, parent link1_2, child link1_3
- added joint joint1_3: type fixed, parent link1_3, child link1_4
- added joint joint1_4: type fixed, parent link1_4, child link1_5
- added joint joint2_1: type fixed, parent link2_1, child link2_2
- added joint joint2_2: type fixed, parent link2_2, child link2_3
- added joint joint2_3: type fixed, parent link2_3, child link2_4
- added joint joint2_4: type fixed, parent link2_4, child link2_5
- added joint joint3_1: type fixed, parent link3_1, child link3_2
- added joint joint3_2: type fixed, parent link3_2, child link3_3
- added joint joint3_3: type fixed, parent link3_3, child link3_4
- added joint joint3_4: type fixed, parent link3_4, child link3_5
- added joint joint4_1: type fixed, parent link4_1, child link4_2
- added joint joint4_2: type fixed, parent link4_2, child link4_3
- added joint joint4_3: type fixed, parent link4_3, child link4_4
- added joint joint4_4: type fixed, parent link4_4, child link4_5
- added joint joint5_1: type fixed, parent link5_1, child link5_2
- added joint joint5_2: type fixed, parent link5_2, child link5_3
- added joint joint5_3: type fixed, parent link5_3, child link5_4
- added joint joint5_4: type fixed, parent link5_4, child link5_5
- added joint joint6_1: type fixed, parent link6_1, child link6_2
- added joint joint6_2: type fixed, parent link6_2, child link6_3
- added joint joint6_3: type fixed, parent link6_3, child link6_4
- added joint joint6_4: type fixed, parent link6_4, child link6_5
- added joint joint7_1: type fixed, parent link7_1, child link7_2
- added joint joint7_2: type fixed, parent link7_2, child link7_3
- added joint joint7_3: type fixed, parent link7_3, child link7_4
- joint joint1: child link1 -> link1_1; parent base -> base2
- joint joint2: child link2 -> link2_1; parent link1 -> link1_5
- joint joint3: child link3 -> link3_1; parent link2 -> link2_5
- joint joint4: child link4 -> link4_1; parent link3 -> link3_5
- joint joint5: child link5 -> link5_1; parent link4 -> link4_5
- joint joint6: child link6 -> link6_1; parent link5 -> link5_5
- joint joint7: child link7 -> link7_1; parent link6 -> link6_5
