Commit message: medio funcionando el virtual robot

File: hermes_virtual_robot/ros/urdf/hermes.urdf (robot description, URDF)
Before this commit: robot HermesRobot, 109 links, 108 joints
Links:
- link l_base: geometry collision mesh filename=package://hermes_virtual_robot/ros/stl/schunk_base1.stl; visual mesh filename=package://hermes_virtual_robot/ros/stl/schunk_base1.stl
- link l_base_hand: geometry collision mesh filename=package://hermes_virtual_robot/ros/stl/left_base_hand.stl; visual mesh filename=package://hermes_virtual_robot/ros/stl/left_base_hand.stl
- link l_base_motor: geometry collision mesh filename=package://hermes_virtual_robot/ros/stl/schunk_base2.stl; visual mesh filename=package://hermes_virtual_robot/ros/stl/schunk_base2.stl
- link l_index1: geometry collision mesh filename=package://hermes_virtual_robot/ros/stl/left_index_link1.stl; visual mesh filename=package://hermes_virtual_robot/ros/stl/left_index_link1.stl
- link l_index2: geometry collision mesh filename=package://hermes_virtual_robot/ros/stl/left_index_link2.stl; visual mesh filename=package://hermes_virtual_robot/ros/stl/left_index_link2.stl
- link l_link1_link: geometry collision mesh filename=package://hermes_virtual_robot/ros/stl/schunk_link1_2.stl; visual mesh filename=package://hermes_virtual_robot/ros/stl/schunk_link1_2.stl
- link l_link1_motor: geometry collision mesh filename=package://hermes_virtual_robot/ros/stl/schunk_link1_1.stl; visual mesh filename=package://hermes_virtual_robot/ros/stl/schunk_link1_1.stl
- link l_link1_motor2: geometry collision mesh filename=package://hermes_virtual_robot/ros/stl/schunk_link1_5.stl; visual mesh filename=package://hermes_virtual_robot/ros/stl/schunk_link1_5.stl
- link l_link1_nbio: geometry collision mesh filename=package://hermes_virtual_robot/ros/stl/schunk_link1_4.stl; visual mesh filename=package://hermes_virtual_robot/ros/stl/schunk_link1_4.stl
- link l_link1_tapa: geometry collision mesh filename=package://hermes_virtual_robot/ros/stl/schunk_link1_3.stl; visual mesh filename=package://hermes_virtual_robot/ros/stl/schunk_link1_3.stl
- link l_link2_link: geometry collision mesh filename=package://hermes_virtual_robot/ros/stl/schunk_link2_2.stl; visual mesh filename=package://hermes_virtual_robot/ros/stl/schunk_link2_2.stl
- link l_link2_motor: geometry collision mesh filename=package://hermes_virtual_robot/ros/stl/schunk_link2_1.stl; visual mesh filename=package://hermes_virtual_robot/ros/stl/schunk_link2_1.stl
- link l_link2_motor2: geometry collision mesh filename=package://hermes_virtual_robot/ros/stl/schunk_link2_5.stl; visual mesh filename=package://hermes_virtual_robot/ros/stl/schunk_link2_5.stl
- link l_link2_nbio: geometry collision mesh filename=package://hermes_virtual_robot/ros/stl/schunk_link2_4.stl; visual mesh filename=package://hermes_virtual_robot/ros/stl/schunk_link2_4.stl
- link l_link2_tapa: geometry collision mesh filename=package://hermes_virtual_robot/ros/stl/schunk_link2_3.stl; visual mesh filename=package://hermes_virtual_robot/ros/stl/schunk_link2_3.stl
- link l_link3_link: geometry collision mesh filename=package://hermes_virtual_robot/ros/stl/schunk_link3_2.stl; visual mesh filename=package://hermes_virtual_robot/ros/stl/schunk_link3_2.stl
- link l_link3_motor: geometry collision mesh filename=package://hermes_virtual_robot/ros/stl/schunk_link3_1.stl; visual mesh filename=package://hermes_virtual_robot/ros/stl/schunk_link3_1.stl
- link l_link3_motor2: geometry collision mesh filename=package://hermes_virtual_robot/ros/stl/schunk_link3_5.stl; visual mesh filename=package://hermes_virtual_robot/ros/stl/schunk_link3_5.stl
- link l_link3_nbio: geometry collision mesh filename=package://hermes_virtual_robot/ros/stl/schunk_link3_4.stl; visual mesh filename=package://hermes_virtual_robot/ros/stl/schunk_link3_4.stl
- link l_link3_tapa: geometry collision mesh filename=package://hermes_virtual_robot/ros/stl/schunk_link3_3.stl; visual mesh filename=package://hermes_virtual_robot/ros/stl/schunk_link3_3.stl
- link l_link4_link: geometry collision mesh filename=package://hermes_virtual_robot/ros/stl/schunk_link4_2.stl; visual mesh filename=package://hermes_virtual_robot/ros/stl/schunk_link4_2.stl
- link l_link4_motor: geometry collision mesh filename=package://hermes_virtual_robot/ros/stl/schunk_link4_1.stl; visual mesh filename=package://hermes_virtual_robot/ros/stl/schunk_link4_1.stl
- link l_link4_motor2: geometry collision mesh filename=package://hermes_virtual_robot/ros/stl/schunk_link4_5.stl; visual mesh filename=package://hermes_virtual_robot/ros/stl/schunk_link4_5.stl
- link l_link4_nbio: geometry collision mesh filename=package://hermes_virtual_robot/ros/stl/schunk_link4_4.stl; visual mesh filename=package://hermes_virtual_robot/ros/stl/schunk_link4_4.stl
- link l_link4_tapa: geometry collision mesh filename=package://hermes_virtual_robot/ros/stl/schunk_link4_3.stl; visual mesh filename=package://hermes_virtual_robot/ros/stl/schunk_link4_3.stl
- link l_link5_link: geometry collision mesh filename=package://hermes_virtual_robot/ros/stl/schunk_link5_2.stl; visual mesh filename=package://hermes_virtual_robot/ros/stl/schunk_link5_2.stl
- link l_link5_motor: geometry collision mesh filename=package://hermes_virtual_robot/ros/stl/schunk_link5_1.stl; visual mesh filename=package://hermes_virtual_robot/ros/stl/schunk_link5_1.stl
- link l_link5_motor2: geometry collision mesh filename=package://hermes_virtual_robot/ros/stl/schunk_link5_5.stl; visual mesh filename=package://hermes_virtual_robot/ros/stl/schunk_link5_5.stl
- link l_link5_nbio: geometry collision mesh filename=package://hermes_virtual_robot/ros/stl/schunk_link5_4.stl; visual mesh filename=package://hermes_virtual_robot/ros/stl/schunk_link5_4.stl
- link l_link5_tapa: geometry collision mesh filename=package://hermes_virtual_robot/ros/stl/schunk_link5_3.stl; visual mesh filename=package://hermes_virtual_robot/ros/stl/schunk_link5_3.stl
- link l_link6_link: geometry collision mesh filename=package://hermes_virtual_robot/ros/stl/schunk_link6_2.stl; visual mesh filename=package://hermes_virtual_robot/ros/stl/schunk_link6_2.stl
- link l_link6_motor: geometry collision mesh filename=package://hermes_virtual_robot/ros/stl/schunk_link6_1.stl; visual mesh filename=package://hermes_virtual_robot/ros/stl/schunk_link6_1.stl
- link l_link6_motor2: geometry collision mesh filename=package://hermes_virtual_robot/ros/stl/schunk_link6_5.stl; visual mesh filename=package://hermes_virtual_robot/ros/stl/schunk_link6_5.stl
- link l_link6_nbio: geometry collision mesh filename=package://hermes_virtual_robot/ros/stl/schunk_link6_4.stl; visual mesh filename=package://hermes_virtual_robot/ros/stl/schunk_link6_4.stl
- link l_link6_tapa: geometry collision mesh filename=package://hermes_virtual_robot/ros/stl/schunk_link6_3.stl; visual mesh filename=package://hermes_virtual_robot/ros/stl/schunk_link6_3.stl
- link l_link7_link: geometry collision mesh filename=package://hermes_virtual_robot/ros/stl/schunk_link7_2.stl; visual mesh filename=package://hermes_virtual_robot/ros/stl/schunk_link7_2.stl
- link l_link7_link2: geometry collision mesh filename=package://hermes_virtual_robot/ros/stl/schunk_link7_4.stl; visual mesh filename=package://hermes_virtual_robot/ros/stl/schunk_link7_4.stl
- link l_link7_motor: geometry collision mesh filename=package://hermes_virtual_robot/ros/stl/schunk_link7_1.stl; visual mesh filename=package://hermes_virtual_robot/ros/stl/schunk_link7_1.stl
- link l_link7_tapa: geometry collision mesh filename=package://hermes_virtual_robot/ros/stl/schunk_link7_3.stl; visual mesh filename=package://hermes_virtual_robot/ros/stl/schunk_link7_3.stl
- link l_middle1: geometry collision mesh filename=package://hermes_virtual_robot/ros/stl/left_middle_link1.stl; visual mesh filename=package://hermes_virtual_robot/ros/stl/left_middle_link1.stl
- link l_middle2: geometry collision mesh filename=package://hermes_virtual_robot/ros/stl/left_middle_link2.stl; visual mesh filename=package://hermes_virtual_robot/ros/stl/left_middle_link2.stl
- link l_pinky1: geometry collision mesh filename=package://hermes_virtual_robot/ros/stl/left_pinky_link1.stl; visual mesh filename=package://hermes_virtual_robot/ros/stl/left_pinky_link1.stl
- link l_pinky2: geometry collision mesh filename=package://hermes_virtual_robot/ros/stl/left_pinky_link2.stl; visual mesh filename=package://hermes_virtual_robot/ros/stl/left_pinky_link2.stl
- link l_ring1: geometry collision mesh filename=package://hermes_virtual_robot/ros/stl/left_ring_link1.stl; visual mesh filename=package://hermes_virtual_robot/ros/stl/left_ring_link1.stl
- link l_ring2: geometry collision mesh filename=package://hermes_virtual_robot/ros/stl/left_ring_link2.stl; visual mesh filename=package://hermes_virtual_robot/ros/stl/left_ring_link2.stl
- link l_thumb1: geometry collision mesh filename=package://hermes_virtual_robot/ros/stl/left_thumb_link1.stl; visual mesh filename=package://hermes_virtual_robot/ros/stl/left_thumb_link1.stl
- link l_thumb2: geometry collision mesh filename=package://hermes_virtual_robot/ros/stl/left_thumb_link2.stl; visual mesh filename=package://hermes_virtual_robot/ros/stl/left_thumb_link2.stl
- link l_thumb3: geometry collision mesh filename=package://hermes_virtual_robot/ros/stl/left_thumb_link3.stl; visual mesh filename=package://hermes_virtual_robot/ros/stl/left_thumb_link3.stl
- link pillar: geometry collision mesh filename=package://hermes_virtual_robot/ros/stl/pillar.stl; visual mesh filename=package://hermes_virtual_robot/ros/stl/pillar.stl
- link r_base: geometry collision mesh filename=package://hermes_virtual_robot/ros/stl/schunk_base1.stl; visual mesh filename=package://hermes_virtual_robot/ros/stl/schunk_base1.stl
- link r_base_hand: geometry collision mesh filename=package://hermes_virtual_robot/ros/stl/right_base_hand.stl; visual mesh filename=package://hermes_virtual_robot/ros/stl/right_base_hand.stl
- link r_base_motor: geometry collision mesh filename=package://hermes_virtual_robot/ros/stl/schunk_base2.stl; visual mesh filename=package://hermes_virtual_robot/ros/stl/schunk_base2.stl
- link r_index1: geometry collision mesh filename=package://hermes_virtual_robot/ros/stl/right_index_link1.stl; visual mesh filename=package://hermes_virtual_robot/ros/stl/right_index_link1.stl
- link r_index2: geometry collision mesh filename=package://hermes_virtual_robot/ros/stl/right_index_link2.stl; visual mesh filename=package://hermes_virtual_robot/ros/stl/right_index_link2.stl
- link r_link1_link: geometry collision mesh filename=package://hermes_virtual_robot/ros/stl/schunk_link1_2.stl; visual mesh filename=package://hermes_virtual_robot/ros/stl/schunk_link1_2.stl
- link r_link1_motor: geometry collision mesh filename=package://hermes_virtual_robot/ros/stl/schunk_link1_1.stl; visual mesh filename=package://hermes_virtual_robot/ros/stl/schunk_link1_1.stl
- link r_link1_motor2: geometry collision mesh filename=package://hermes_virtual_robot/ros/stl/schunk_link1_5.stl; visual mesh filename=package://hermes_virtual_robot/ros/stl/schunk_link1_5.stl
- link r_link1_nbio: geometry collision mesh filename=package://hermes_virtual_robot/ros/stl/schunk_link1_4.stl; visual mesh filename=package://hermes_virtual_robot/ros/stl/schunk_link1_4.stl
- link r_link1_tapa: geometry collision mesh filename=package://hermes_virtual_robot/ros/stl/schunk_link1_3.stl; visual mesh filename=package://hermes_virtual_robot/ros/stl/schunk_link1_3.stl
- link r_link2_link: geometry collision mesh filename=package://hermes_virtual_robot/ros/stl/schunk_link2_2.stl; visual mesh filename=package://hermes_virtual_robot/ros/stl/schunk_link2_2.stl
- link r_link2_motor: geometry collision mesh filename=package://hermes_virtual_robot/ros/stl/schunk_link2_1.stl; visual mesh filename=package://hermes_virtual_robot/ros/stl/schunk_link2_1.stl
- link r_link2_motor2: geometry collision mesh filename=package://hermes_virtual_robot/ros/stl/schunk_link2_5.stl; visual mesh filename=package://hermes_virtual_robot/ros/stl/schunk_link2_5.stl
- link r_link2_nbio: geometry collision mesh filename=package://hermes_virtual_robot/ros/stl/schunk_link2_4.stl; visual mesh filename=package://hermes_virtual_robot/ros/stl/schunk_link2_4.stl
- link r_link2_tapa: geometry collision mesh filename=package://hermes_virtual_robot/ros/stl/schunk_link2_3.stl; visual mesh filename=package://hermes_virtual_robot/ros/stl/schunk_link2_3.stl
- link r_link3_link: geometry collision mesh filename=package://hermes_virtual_robot/ros/stl/schunk_link3_2.stl; visual mesh filename=package://hermes_virtual_robot/ros/stl/schunk_link3_2.stl
- link r_link3_motor: geometry collision mesh filename=package://hermes_virtual_robot/ros/stl/schunk_link3_1.stl; visual mesh filename=package://hermes_virtual_robot/ros/stl/schunk_link3_1.stl
- link r_link3_motor2: geometry collision mesh filename=package://hermes_virtual_robot/ros/stl/schunk_link3_5.stl; visual mesh filename=package://hermes_virtual_robot/ros/stl/schunk_link3_5.stl
- link r_link3_nbio: geometry collision mesh filename=package://hermes_virtual_robot/ros/stl/schunk_link3_4.stl; visual mesh filename=package://hermes_virtual_robot/ros/stl/schunk_link3_4.stl
- link r_link3_tapa: geometry collision mesh filename=package://hermes_virtual_robot/ros/stl/schunk_link3_3.stl; visual mesh filename=package://hermes_virtual_robot/ros/stl/schunk_link3_3.stl
- link r_link4_link: geometry collision mesh filename=package://hermes_virtual_robot/ros/stl/schunk_link4_2.stl; visual mesh filename=package://hermes_virtual_robot/ros/stl/schunk_link4_2.stl
- link r_link4_motor: geometry collision mesh filename=package://hermes_virtual_robot/ros/stl/schunk_link4_1.stl; visual mesh filename=package://hermes_virtual_robot/ros/stl/schunk_link4_1.stl
- link r_link4_motor2: geometry collision mesh filename=package://hermes_virtual_robot/ros/stl/schunk_link4_5.stl; visual mesh filename=package://hermes_virtual_robot/ros/stl/schunk_link4_5.stl
- link r_link4_nbio: geometry collision mesh filename=package://hermes_virtual_robot/ros/stl/schunk_link4_4.stl; visual mesh filename=package://hermes_virtual_robot/ros/stl/schunk_link4_4.stl
- link r_link4_tapa: geometry collision mesh filename=package://hermes_virtual_robot/ros/stl/schunk_link4_3.stl; visual mesh filename=package://hermes_virtual_robot/ros/stl/schunk_link4_3.stl
- link r_link5_link: geometry collision mesh filename=package://hermes_virtual_robot/ros/stl/schunk_link5_2.stl; visual mesh filename=package://hermes_virtual_robot/ros/stl/schunk_link5_2.stl
- link r_link5_motor: geometry collision mesh filename=package://hermes_virtual_robot/ros/stl/schunk_link5_1.stl; visual mesh filename=package://hermes_virtual_robot/ros/stl/schunk_link5_1.stl
- link r_link5_motor2: geometry collision mesh filename=package://hermes_virtual_robot/ros/stl/schunk_link5_5.stl; visual mesh filename=package://hermes_virtual_robot/ros/stl/schunk_link5_5.stl
- link r_link5_nbio: geometry collision mesh filename=package://hermes_virtual_robot/ros/stl/schunk_link5_4.stl; visual mesh filename=package://hermes_virtual_robot/ros/stl/schunk_link5_4.stl
- link r_link5_tapa: geometry collision mesh filename=package://hermes_virtual_robot/ros/stl/schunk_link5_3.stl; visual mesh filename=package://hermes_virtual_robot/ros/stl/schunk_link5_3.stl
- link r_link6_link: geometry collision mesh filename=package://hermes_virtual_robot/ros/stl/schunk_link6_2.stl; visual mesh filename=package://hermes_virtual_robot/ros/stl/schunk_link6_2.stl
- link r_link6_motor: geometry collision mesh filename=package://hermes_virtual_robot/ros/stl/schunk_link6_1.stl; visual mesh filename=package://hermes_virtual_robot/ros/stl/schunk_link6_1.stl
- link r_link6_motor2: geometry collision mesh filename=package://hermes_virtual_robot/ros/stl/schunk_link6_5.stl; visual mesh filename=package://hermes_virtual_robot/ros/stl/schunk_link6_5.stl
- link r_link6_nbio: geometry collision mesh filename=package://hermes_virtual_robot/ros/stl/schunk_link6_4.stl; visual mesh filename=package://hermes_virtual_robot/ros/stl/schunk_link6_4.stl
- link r_link6_tapa: geometry collision mesh filename=package://hermes_virtual_robot/ros/stl/schunk_link6_3.stl; visual mesh filename=package://hermes_virtual_robot/ros/stl/schunk_link6_3.stl
- link r_link7_link: geometry collision mesh filename=package://hermes_virtual_robot/ros/stl/schunk_link7_2.stl; visual mesh filename=package://hermes_virtual_robot/ros/stl/schunk_link7_2.stl
- link r_link7_link2: geometry collision mesh filename=package://hermes_virtual_robot/ros/stl/schunk_link7_4.stl; visual mesh filename=package://hermes_virtual_robot/ros/stl/schunk_link7_4.stl
- link r_link7_motor: geometry collision mesh filename=package://hermes_virtual_robot/ros/stl/schunk_link7_1.stl; visual mesh filename=package://hermes_virtual_robot/ros/stl/schunk_link7_1.stl
- link r_link7_tapa: geometry collision mesh filename=package://hermes_virtual_robot/ros/stl/schunk_link7_3.stl; visual mesh filename=package://hermes_virtual_robot/ros/stl/schunk_link7_3.stl
- link r_middle1: geometry collision mesh filename=package://hermes_virtual_robot/ros/stl/right_middle_link1.s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; visual mesh filename=package://hermes_virtual_robot/ros/stl/right_middle_link1.s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
- link r_middle2: geometry collision mesh filename=package://hermes_virtual_robot/ros/stl/right_middle_link2.s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; visual mesh filename=package://hermes_virtual_robot/ros/stl/right_middle_link2.s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
- link r_pinky1: geometry collision mesh filename=package://hermes_virtual_robot/ros/stl/right_pinky_link1.stl; visual mesh filename=package://hermes_virtual_robot/ros/stl/right_pinky_link1.stl
- link r_pinky2: geometry collision mesh filename=package://hermes_virtual_robot/ros/stl/right_pinky_link2.stl; visual mesh filename=package://hermes_virtual_robot/ros/stl/right_pinky_link2.stl
- link r_ring1: geometry collision mesh filename=package://hermes_virtual_robot/ros/stl/right_ring_link1.stl; visual mesh filename=package://hermes_virtual_robot/ros/stl/right_ring_link1.stl
- link r_ring2: geometry collision mesh filename=package://hermes_virtual_robot/ros/stl/right_ring_link2.stl; visual mesh filename=package://hermes_virtual_robot/ros/stl/right_ring_link2.stl
- link r_thumb1: geometry collision mesh filename=package://hermes_virtual_robot/ros/stl/right_thumb_link1.stl; visual mesh filename=package://hermes_virtual_robot/ros/stl/right_thumb_link1.stl
- link r_thumb2: geometry collision mesh filename=package://hermes_virtual_robot/ros/stl/right_thumb_link2.stl; visual mesh filename=package://hermes_virtual_robot/ros/stl/right_thumb_link2.stl
- link r_thumb3: geometry collision mesh filename=package://hermes_virtual_robot/ros/stl/right_thumb_link3.stl; visual mesh filename=package://hermes_virtual_robot/ros/stl/right_thumb_link3.stl
